File: CAN-breakout-3.3V-v3.brd (EAGLE design)
At the start: 27.3 x 15.2 mm, 10 parts, among them IC1 SN65HVD232

Commit message: Create Gerbers
Parts:
- removed U$3: SPARK_LOGO2, Spark:SPARK_LOGO2
Other:
- board text added: "(Do not populate)"
- board text added: "All components go on top"
- board text added: "C1"
- board text added: "C2"
- board text added: "Carloop"
- board text added: "IC1"
- board text added: "JP1"
- board text added: "JP2"
- board text added: "JP3"
- board text added: "JP4"
- board text added: "Made by"
- board text added: "R1"
- board text added: "R2"
- board text added: "carloop.io"
- board text removed: "Particle pins RX=D2 TX=D1"
